File: BME280-env-sensor-breakout-module.kicad_sch (KiCad schematic)
At the start: 0 parts

Commit message: completed schematic and routing
Parts:
- added C1, C2: 100nF, Capacitor_SMD:C_0603_1608Metric_Pad1.08x0.95mm_HandSolder, symbol Device:C
- added J1: I2C_HEADER, Connector_PinHeader_2.54mm:PinHeader_1x04_P2.54mm_Vertical, symbol Connector:Conn_01x04_Pin
- added R1, R2: 2.2K, Resistor_SMD:R_0603_1608Metric_Pad0.98x0.95mm_HandSolder, symbol Device:R
- added U1: BME280, BME280:PSON65P250X250X100-8N, symbol BME280:BME280
Connections:
- new net +3.3V: C1.1, C2.1, J1.1 (Pin_1), R1.1, R2.1, U1.2 (CSB), U1.5 (SDO), U1.6 (VDDIO), U1.8 (VDD)
- new net GND: C1.2, C2.2, J1.3 (Pin_3), U1.1 (GND), U1.7 (GND)
- new net SCK: J1.2 (Pin_2), R2.2, U1.4 (SCK)
- new net SDA: J1.4 (Pin_4), R1.2, U1.3 (SDI)
Other:
- note added: "Design Choices I2C MODE: CSB tied to VDDIO SDO to VDDIO: Slave Address LSB = 1 I2C Standard Mode(100KHz) = 2.2K Ohm Pull Ups Filter caps = 100nF recommended by datasheet"
- company: (none) -> HTronics
- title: (none) -> BME280 Breakout Module
